Commit message: Updated drone's urdf.

File: urdf/drone/gimbal.transmission.urdf.xacro (robot description, xacro)
@@ -7,5 +7,5 @@
         </actuator>
         <joint name="yaw_joint">
-            <offset>5.20927</offset>
+            <offset>5.182</offset>
             <hardwareInterface>hardware_interface/EffortJointInterface</hardwareInterface>
         </joint>
@@ -17,5 +17,5 @@
         </actuator>
         <joint name="pitch_joint">
-            <offset>0.887</offset>
+            <offset>0.9267</offset>
             <hardwareInterface>hardware_interface/EffortJointInterface</hardwareInterface>
         </joint>

File: urdf/drone/gimbal.urdf.xacro (robot description, xacro)
@@ -2,8 +2,8 @@
 <robot xmlns:xacro="http://www.ros.org/wiki/xacro">
     <xacro:property name="threshold" value="0.1"/>
-    <xacro:property name="pitch_lower_limit" value="-0.6"/>
-    <xacro:property name="pitch_upper_limit" value="0.457"/>
-    <xacro:property name="yaw_lower_limit" value="-0.627"/>
-    <xacro:property name="yaw_upper_limit" value="0.627"/>
+    <xacro:property name="pitch_lower_limit" value="-0.406"/>
+    <xacro:property name="pitch_upper_limit" value="0.867"/>
+    <xacro:property name="yaw_lower_limit" value="-1.288"/>
+    <xacro:property name="yaw_upper_limit" value="1.138"/>
     <link name="yaw">
         <inertial>

File: urdf/drone/shooter.transmission.urdf.xacro (robot description, xacro)
@@ -14,5 +14,5 @@
         <type>transmission_interface/SimpleTransmission</type>
         <actuator name="left_friction_wheel_joint_motor">
-            <mechanicalReduction>-1</mechanicalReduction>
+            <mechanicalReduction>1</mechanicalReduction>
         </actuator>
         <joint name="left_friction_wheel_joint">
@@ -23,5 +23,5 @@
         <type>transmission_interface/SimpleTransmission</type>
         <actuator name="right_friction_wheel_joint_motor">
-            <mechanicalReduction>-1</mechanicalReduction>
+            <mechanicalReduction>1</mechanicalReduction>
         </actuator>
         <joint name="right_friction_wheel_joint">

Commit message: Updated drone's urdf.

File: urdf/drone/gimbal.transmission.urdf.xacro (robot description, xacro)
@@ -7,5 +7,5 @@
         </actuator>
         <joint name="yaw_joint">
-            <offset>5.182</offset>
+            <offset>5.1502</offset>
             <hardwareInterface>hardware_interface/EffortJointInterface</hardwareInterface>
         </joint>

File: urdf/drone/gimbal.urdf.xacro (robot description, xacro)
@@ -1,5 +1,6 @@
 <?xml version="1.0" encoding="utf-8"?>
 <robot xmlns:xacro="http://www.ros.org/wiki/xacro">
-    <xacro:property name="threshold" value="0.1"/>
+    <xacro:property name="threshold_pitch" value="0.1"/>
+    <xacro:property name="threshold_yaw" value="0.12"/>
     <xacro:property name="pitch_lower_limit" value="-0.406"/>
     <xacro:property name="pitch_upper_limit" value="0.867"/>
@@ -30,8 +31,8 @@
                 rpy="0 0 0"/>
         <dynamics damping="0.0" friction="0.1"/>
-        <limit effort="1.2" velocity="31" lower="-1e10" upper="1e10"/>
+        <limit effort="1.2" velocity="31" lower="${yaw_lower_limit}" upper="${yaw_upper_limit}"/>
         <safety_controller k_position="100" k_velocity="0.1"
-                           soft_lower_limit="${yaw_lower_limit+threshold}"
-                           soft_upper_limit="${yaw_upper_limit-threshold}"/>
+                           soft_lower_limit="${yaw_lower_limit+threshold_yaw}"
+                           soft_upper_limit="${yaw_upper_limit-threshold_yaw}"/>
         <parent link="base_link"/>
         <child link="yaw"/>
@@ -63,6 +64,6 @@
         <limit effort="3.0" velocity="86" lower="${pitch_lower_limit}" upper="${pitch_upper_limit}"/>
         <safety_controller k_position="100" k_velocity="0.1"
-                           soft_lower_limit="${pitch_lower_limit+threshold}"
-                           soft_upper_limit="${pitch_upper_limit-threshold}"/>
+                           soft_lower_limit="${pitch_lower_limit+threshold_pitch}"
+                           soft_upper_limit="${pitch_upper_limit-threshold_pitch}"/>
         <parent link="yaw"/>
         <child link="pitch"/>

Commit message: Updated drone's config.

File: urdf/drone/gimbal.transmission.urdf.xacro (robot description, xacro)
@@ -7,5 +7,5 @@
         </actuator>
         <joint name="yaw_joint">
-            <offset>5.1502</offset>
+            <offset>1.825</offset>
             <hardwareInterface>hardware_interface/EffortJointInterface</hardwareInterface>
         </joint>

File: urdf/drone/gimbal.urdf.xacro (robot description, xacro)
@@ -1,10 +1,9 @@
 <?xml version="1.0" encoding="utf-8"?>
 <robot xmlns:xacro="http://www.ros.org/wiki/xacro">
-    <xacro:property name="threshold_pitch" value="0.1"/>
-    <xacro:property name="threshold_yaw" value="0.12"/>
-    <xacro:property name="pitch_lower_limit" value="-0.406"/>
-    <xacro:property name="pitch_upper_limit" value="0.867"/>
-    <xacro:property name="yaw_lower_limit" value="-1.1917"/>
-    <xacro:property name="yaw_upper_limit" value="1.138"/>
+    <xacro:property name="threshold" value="0.1"/>
+    <xacro:property name="pitch_lower_limit" value="-0.15"/>
+    <xacro:property name="pitch_upper_limit" value="0.62"/>
+    <xacro:property name="yaw_lower_limit" value="-1.36"/>
+    <xacro:property name="yaw_upper_limit" value="0.868"/>
     <link name="yaw">
         <inertial>
@@ -33,6 +32,6 @@
         <limit effort="1.2" velocity="31" lower="${yaw_lower_limit}" upper="${yaw_upper_limit}"/>
         <safety_controller k_position="100" k_velocity="0.1"
-                           soft_lower_limit="${yaw_lower_limit+threshold_yaw}"
-                           soft_upper_limit="${yaw_upper_limit-threshold_yaw}"/>
+                           soft_lower_limit="${yaw_lower_limit+threshold}"
+                           soft_upper_limit="${yaw_upper_limit-threshold}"/>
         <parent link="base_link"/>
         <child link="yaw"/>
@@ -64,6 +63,6 @@
         <limit effort="3.0" velocity="86" lower="${pitch_lower_limit}" upper="${pitch_upper_limit}"/>
         <safety_controller k_position="100" k_velocity="0.1"
-                           soft_lower_limit="${pitch_lower_limit+threshold_pitch}"
-                           soft_upper_limit="${pitch_upper_limit-threshold_pitch}"/>
+                           soft_lower_limit="${pitch_lower_limit+threshold}"
+                           soft_upper_limit="${pitch_upper_limit-threshold}"/>
         <parent link="yaw"/>
         <child link="pitch"/>
