Commit message: Updated config and urdf.

File: urdf/hero/gimbal.transmission.urdf.xacro (robot description, xacro)
@@ -7,5 +7,5 @@
         </actuator>
         <joint name="yaw_joint">
-            <offset>-0.561505488</offset>
+            <offset>6.998109012</offset>
             <hardwareInterface>hardware_interface/EffortJointInterface</hardwareInterface>
         </joint>
@@ -17,5 +17,5 @@
         </actuator>
         <joint name="pitch_joint">
-            <offset>2.180819812</offset>
+            <offset>2.090819812</offset>
             <hardwareInterface>hardware_interface/EffortJointInterface</hardwareInterface>
         </joint>

File: urdf/hero/hero.urdf.xacro (robot description, xacro)
@@ -16,10 +16,12 @@
             <xacro:include filename="$(find rm_description)/urdf/common/imu.urdf.xacro"/>
             <xacro:include filename="$(find rm_description)/urdf/common/camera.urdf.xacro"/>
-            <xacro:camera_sensor xyz="0.0445 0 0.109" rpy="${pi} 0 -0.02" frame_id="$(arg camera_link)" parent="pitch"
+            <xacro:camera_sensor xyz="0.098768 0.0 0.273105" rpy="${pi} 3.0545 ${pi}" frame_id="$(arg camera_link)"
+                                 parent="pitch"
                                  camera_sim="$(arg use_simulation)"/>
-            <xacro:camera_optical_frame xyz="0.105 0.0071 0.13" rpy="-1.5786 -0.0025 -1.570"
+            <xacro:camera_optical_frame xyz="0.0831144205203709 -0.044000480243231284 0.2839307026247077"
+                                        rpy="-1.8177988 0.1017211 -1.5986981"
                                         frame_id="$(arg camera_optical_frame)" parent="pitch"
                                         camera_sim="$(arg use_simulation)"/>
-            <xacro:IMU connected_to="pitch" imu_name="gimbal_imu" xyz="0.08 0. 0.08" rpy="${pi} 0 ${pi/2}"/>
+            <xacro:IMU connected_to="pitch" imu_name="gimbal_imu" xyz="0.08 0. 0.08" rpy="0 0 -${pi/2}"/>
             <xacro:if value="$(arg load_shooter)">
                 <xacro:include filename="$(find rm_description)/urdf/hero/shooter.urdf.xacro"/>

File: urdf/hero/shooter.urdf.xacro (robot description, xacro)
@@ -33,5 +33,5 @@
         <origin xyz="0 0 0.0223" rpy="0 0 0"/>
         <dynamics damping="0.0" friction="0.01"/>
-        <limit effort="18" velocity="13.5327" lower="-1e16" upper="1e16"/>
+        <limit effort="5" velocity="50" lower="-1e16" upper="1e16"/>
         <parent link="base_link"/>
         <child link="trigger"/>

File: urdf/little_standard/gimbal.transmission.urdf.xacro (robot description, xacro)
@@ -1,29 +1,31 @@
 <?xml version="1.0" encoding="utf-8"?>
 <robot>
-    <transmission name="trans_trigger_joint">
+    <transmission name="trans_yaw_joint">
         <type>transmission_interface/SimpleTransmission</type>
-        <actuator name="trigger_joint_motor">
-            <mechanicalReduction>19.2032</mechanicalReduction>
-        </actuator>
-        <joint name="trigger_joint">
-            <hardwareInterface>hardware_interface/EffortJointInterface</hardwareInterface>
-            <offset>0.5</offset>
-        </joint>
-    </transmission>
-    <transmission name="trans_left_friction_wheel_joint">
-        <type>transmission_interface/SimpleTransmission</type>
-        <actuator name="left_friction_wheel_joint_motor">
+        <actuator name="yaw_joint_motor">
             <mechanicalReduction>1</mechanicalReduction>
         </actuator>
-        <joint name="left_friction_wheel_joint">
+        <joint name="yaw_joint">
+            <offset>-5.01021</offset>
             <hardwareInterface>hardware_interface/EffortJointInterface</hardwareInterface>
         </joint>
     </transmission>
-    <transmission name="trans_right_friction_wheel_joint">
+    <transmission name="trans_pitch_joint">
         <type>transmission_interface/SimpleTransmission</type>
-        <actuator name="right_friction_wheel_joint_motor">
-            <mechanicalReduction>1</mechanicalReduction>
+        <actuator name="pitch_joint_motor">
+            <mechanicalReduction>-1</mechanicalReduction>
         </actuator>
-        <joint name="right_friction_wheel_joint">
+        <joint name="pitch_joint">
+            <offset>3.5116</offset>
+            <hardwareInterface>hardware_interface/EffortJointInterface</hardwareInterface>
+        </joint>
+    </transmission>
+    <transmission name="trans_cover_joint">
+        <type>transmission_interface/SimpleTransmission</type>
+        <actuator name="cover_joint_motor">
+            <mechanicalReduction>-1</mechanicalReduction>
+        </actuator>
+        <joint name="cover_joint">
+            <offset>0</offset>
             <hardwareInterface>hardware_interface/EffortJointInterface</hardwareInterface>
         </joint>

File: urdf/little_standard/shooter.transmission.urdf.xacro (robot description, xacro)
@@ -4,9 +4,9 @@
         <type>transmission_interface/SimpleTransmission</type>
         <actuator name="trigger_joint_motor">
-            <mechanicalReduction>19.2032</mechanicalReduction>
+            <mechanicalReduction>1</mechanicalReduction>
         </actuator>
         <joint name="trigger_joint">
             <hardwareInterface>hardware_interface/EffortJointInterface</hardwareInterface>
-            <offset>0.5</offset>
+            <offset>0.2</offset>
         </joint>
     </transmission>
